Commit message: Update my_robot.xacro

File: catkin_ws/src/my_robot/urdf/my_robot.xacro (robot description, xacro)
@@ -4,4 +4,7 @@
   <material name="Green">
     <color rgba=" 0 0.9 0 1"/>
+  </material>
+  <material name="Blue">
+    <color rgba=" 0 0 0.9 1"/>
   </material>
   <link name="robot_footprint"></link>
@@ -183,3 +186,9 @@
     <material>Gazebo/Green</material>
   </gazebo>
+  <gazebo reference="SIDE_left_wheel">
+    <material>Gazebo/Blue</material>
+  </gazebo>
+  <gazebo reference="SIDE_right_wheel">
+    <material>Gazebo/Blue</material>
+  </gazebo>
 </robot>
